File: board_files/one_channel_amplifier/one_channel_amplifier.kicad_pcb (KiCad board)
At the start: 2 copper layers, 25 parts, among them J1 Screw_Terminal_01x03, J2 Conn_01x02, J3 Conn_01x02, J4 Screw_Terminal_01x02, U1 LM3886

Commit message: Initial component placement process
Parts:
- added J5: Conn_01x02, Connector_PinHeader_2.54mm:PinHeader_1x02_P2.54mm_Vertical, F.Cu at (175.0, 92.2)
- added J6: Screw_Terminal_01x02, TerminalBlock:TerminalBlock_bornier-2_P5.08mm, F.Cu at (120.9, 79.2)
- C11: value 100uF -> 0.1uF; footprint Capacitor_THT:CP_Radial_D8.0mm_P3.50mm -> Capacitor_SMD:C_0603_1608Metric
- C2: value 470uF -> 22uF; footprint Capacitor_THT:CP_Radial_D16.0mm_P7.50mm -> Capacitor_THT:CP_Radial_D10.0mm_P5.00mm
- C3: value 22uF -> 4.7uF; footprint Capacitor_THT:CP_Radial_D10.0mm_P5.00mm -> Resistor_SMD:R_1210_3225Metric
- C4: value 22uF -> 470uF; footprint Capacitor_THT:CP_Radial_D10.0mm_P5.00mm -> Capacitor_THT:CP_Radial_D16.0mm_P7.50mm
- C5: value 4.7uF -> 22uF; footprint Resistor_SMD:R_1210_3225Metric -> Capacitor_THT:CP_Radial_D10.0mm_P5.00mm
- C7: value 1500pF -> 100uF; footprint Capacitor_SMD:C_0603_1608Metric -> Capacitor_THT:CP_Radial_D8.0mm_P3.50mm
- C8: value 0.1uF -> 220pF
- C9: value 220pF -> 1500pF
- J1: value Screw_Terminal_01x03 -> Screw_Terminal_01x02; footprint TerminalBlock:TerminalBlock_bornier-3_P5.08mm -> Connector_QC_Blade_User:TE_QC_250_Male_Blade_P5.08
- J2, J3: value Conn_01x02 -> Screw_Terminal_01x02; footprint Connector_PinHeader_2.54mm:PinHeader_1x02_P2.54mm_Vertical -> Connector_QC_Blade_User:TE_QC_250_Male_Blade_P5.08
- J4: value Screw_Terminal_01x02 -> Conn_01x02; footprint TerminalBlock:TerminalBlock_bornier-2_P5.08mm -> Connector_PinHeader_2.54mm:PinHeader_1x02_P2.54mm_Vertical
- R1: value 1k -> 63.4k
- R2: value 6.34k -> 1k
- R3: value 63.4k -> 2.7
- R6: value 2.7 -> 6.34k
- moved C7 110.3 mm to (171.4, 82.8)
- moved C9 106.9 mm to (169.9, 91.7)
- moved C1 104.0 mm to (148.3, 110.2)
- moved U1 95.6 mm to (143.9, 85.9)
- moved C10 93.7 mm to (159.4, 61.9)
- moved C12 93.7 mm to (155.4, 64.4)
- moved R7 93.7 mm to (174.6, 55.9)
- moved R5 93.7 mm to (167.4, 61.9)
- moved R6 93.7 mm to (163.4, 64.4)
- moved R2 90.5 mm to (169.9, 90.2)
- moved C8 90.3 mm to (166.9, 90.9), turned to 90 degrees
- moved L1 85.8 mm to (130.8, 79.0), turned to 180 degrees
- moved C5 74.8 mm to (132.1, 92.5), turned to 90 degrees
- moved R1 71.8 mm to (165.9, 81.3)
- moved C2 71.7 mm to (149.6, 96.3)
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Connections:
- C2 pad 1: GND -> VCC
- C2 pad 2: VEE -> GND
- C5 pad 1: VCC -> GND
- C5 pad 2: GND -> VEE
- C8 pad 1: Net-(C8-Pad1) -> Net-(C10-Pad1)
- C8 pad 2: GND -> Net-(C8-Pad2)
- C9 pad 1: Net-(C10-Pad1) -> Net-(C8-Pad2)
- C9 pad 2: Net-(C7-Pad1) -> GND
- J1 pad 1: VEE -> VCC
- J1 pad 2: GND -> VCC
- J2 pad 2: Net-(J2-Pad2) -> GND
- J3 pad 1: Net-(J3-Pad1) -> VEE
- J4 pad 2: GND -> VEE
- L1 pad 2: Net-(J4-Pad1) -> Net-(J6-Pad1)
- R1 pad 2: Net-(J2-Pad2) -> Net-(J4-Pad1)
- R2 pad 1: Net-(C10-Pad1) -> Net-(C8-Pad2)
- R2 pad 2: Net-(C8-Pad1) -> Net-(J5-Pad2)
- R3 pad 1: Net-(C11-Pad1) -> Net-(L1-Pad1)
- R3 pad 2: Net-(J3-Pad1) -> Net-(J6-Pad1)
- R6 pad 1: Net-(L1-Pad1) -> Net-(C10-Pad1)
- R6 pad 2: Net-(C12-Pad1) -> Net-(C11-Pad1)
- R7 pad 2: Net-(J4-Pad1) -> Net-(C12-Pad1)
- U1 pad 10: Net-(C7-Pad1) -> Net-(C8-Pad2)
- U1 pad 8: Net-(C11-Pad1) -> Net-(C7-Pad1)
Other:
- board outline added: 50.8 x 50.8 mm
